Commit message: lidar

File: src/simulator/sitl/yutu_description/urdf/urdf/YuTuURDF.urdf (robot description, URDF)
Before this commit: robot yutu_description, 13 links, 12 joints
Links:
- removed link lidar_Link
- added link laser_Link, mass 0.001; collision mesh filename=package://yutu_description/meshes/laser_Link.STL; visual mesh filename=package://yutu_description/meshes/laser_Link.STL
Joints:
- removed joint lidar_joint
- added joint laser_joint: type fixed, parent base_link, child laser_Link, origin xyz=0.393474958757372 0.00225655709560415 0.67 rpy=0 0 0, axis 0 0 0

File: src/simulator/sitl/yutu_description/urdf/xacro/2d_laser.xacro (robot description, xacro)
@@ -2,6 +2,6 @@
 <robot xmlns:xacro="http://www.ros.org/wiki/xacro" name="velodyne">
   <!-- Gazebo requires the velodyne_gazebo_plugins package -->
-  <gazebo reference="lidar_link">
-		<sensor type="ray" name="rplidar">
+  <gazebo reference="laser_link">
+		<sensor type="ray" name="rplaser">
       <pose>0 0 0 0 0 0</pose>
       <visualize>true</visualize>
@@ -27,7 +27,7 @@
         </noise>
       </ray>
-      <plugin name="gazebo_rplidar" filename="libgazebo_ros_laser.so">
+      <plugin name="gazebo_rplaser" filename="libgazebo_ros_laser.so">
         <topicName>scan</topicName>
-        <frameName>$(arg ns)/lidar_link</frameName>
+        <frameName>$(arg ns)/laser_link</frameName>
       </plugin>
     </sensor>

File: src/simulator/sitl/yutu_description/urdf/xacro/sensor.xacro (robot description, xacro)
@@ -128,5 +128,5 @@
 		</sensor>
 	</gazebo>
-    <!-- <gazebo reference="lidar_Link">
+    <!-- <gazebo reference="laser_Link">
 		<sensor type="ray" name="head_hokuyo_sensor">
 			<pose>0 0 0 0 0 0</pose>
@@ -155,10 +155,10 @@
 			<plugin name="gazebo_ros_head_hokuyo_controller" filename="libgazebo_ros_laser.so">
 				<topicName>laser/scan</topicName>
-				<frameName>lidar_Link</frameName>
+				<frameName>laser_Link</frameName>
 			</plugin>
 		</sensor>
 	</gazebo> -->
-	<gazebo reference="lidar_Link">
-		<sensor type="ray" name="rplidar">
+	<gazebo reference="laser_Link">
+		<sensor type="ray" name="rplaser">
 			<pose>0 0 0 0 0 0</pose>
 			<visualize>false</visualize>
@@ -184,7 +184,7 @@
 				</noise>
 			</ray>
-			<plugin name="gazebo_rplidar" filename="libgazebo_ros_laser.so">
+			<plugin name="gazebo_rplaser" filename="libgazebo_ros_laser.so">
 				<topicName>/scan</topicName>
-				<frameName>lidar_Link</frameName>
+				<frameName>laser_Link</frameName>
 			</plugin>
 		</sensor>

File: src/simulator/sitl/yutu_description/urdf/xacro/velodyne.xacro (robot description, xacro)
@@ -2,6 +2,6 @@
 <robot xmlns:xacro="http://www.ros.org/wiki/xacro" name="velodyne">
     <!-- Gazebo requires the velodyne_gazebo_plugins package -->
-    <gazebo reference="lidar_link">
-		<sensor name='3d_lidar' type='gpu_ray'>
+    <gazebo reference="laser_link">
+		<sensor name='3d_laser' type='gpu_ray'>
 			<ray>
 				<scan>
@@ -26,5 +26,5 @@
 			<plugin name='3d_laser' filename='libgazebo_ros_velodyne_gpu_laser.so'>
 				<topicName>/velodyne_points</topicName>
-				<frameName>lidar_link</frameName>
+				<frameName>laser_link</frameName>
 				<gaussianNoise>0.008</gaussianNoise>
 			</plugin>

File: src/simulator/sitl/yutu_description/urdf/xacro/yutu_sim.xacro (robot description, xacro)
@@ -110,5 +110,5 @@
   </joint>
   <link
-    name="lidar_link">
+    name="laser_link">
     <inertial>
       <origin
@@ -131,5 +131,5 @@
       <geometry>
         <mesh
-          filename="package://yutu_description/meshes/lidar_link.STL" />
+          filename="package://yutu_description/meshes/laser_link.STL" />
       </geometry>
       <material
@@ -145,10 +145,10 @@
       <geometry>
         <mesh
-          filename="package://yutu_description/meshes/lidar_link.STL" />
-      </geometry>
-    </collision>
-  </link>
-  <joint
-    name="lidar_joint"
+          filename="package://yutu_description/meshes/laser_link.STL" />
+      </geometry>
+    </collision>
+  </link>
+  <joint
+    name="laser_joint"
     type="fixed">
     <origin
@@ -158,5 +158,5 @@
       link="base_link" />
     <child
-      link="lidar_link" />
+      link="laser_link" />
     <axis
       xyz="0 0 0" />
